File: src/HardwareDesign/1.0.0/usb_interface.kicad_sch (KiCad schematic)
At the start: 31 parts, among them IC7 TPS74801DRCT, IC8 SN74LVC1G97QDCKRQ1, IC9 FSUSB42MUX, J3 USB-TYPE-C-018

Commit message: update design
Parts:
- removed C54: 1uF 50V, Capacitor_SMD:C_0402_1005Metric, symbol DS_Capacitor_0402:1uF 50V 0402
- added C54: 4.7uF 25V, Capacitor_SMD:C_0402_1005Metric, symbol DS_Capacitor_0402:4.7uF 25V 0402
Connections:
- net BIAS is gone; now on net +5V: IC7.4 (BIAS)
- net +5V: now also C54.1
- net GND: now also C54.2
Changed lines of the file:
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@@
 	)
 	(junction
+		(at 120.65 90.17)
+		(diameter 0)
+		(color 0 0 0 0)
+	)
+	(junction
 		(at 143.51 172.72)
 		(diameter 0)
@@
 	)
 	(junction
+		(at 120.65 95.25)
+		(diameter 0)
+		(color 0 0 0 0)
+	)
+	(junction
 		(at 74.93 213.36)
 		(diameter 0)
@@
 	(wire
 		(pts
+			(xy 120.65 90.17) (xy 120.65 95.25)
+		)
+		(stroke
+			(width 0)
+			(type default)
+		)
+	)
+	(wire
+		(pts
 			(xy 38.1 223.52) (xy 50.8 223.52)
 		)
@@
 	(wire
 		(pts
-			(xy 92.71 95.25) (xy 124.46 95.25)
+			(xy 92.71 95.25) (xy 120.65 95.25)
 		)
 		(stroke
@@
 	(wire
 		(pts
+			(xy 120.65 95.25) (xy 124.46 95.25)
+		)
+		(stroke
+			(width 0)
+			(type default)
+		)
+	)
+	(wire
+		(pts
 			(xy 120.65 87.63) (xy 120.65 90.17)
 		)
@@
 		)
 	)
-	(label "BIAS"
-		(at 116.84 95.25 0)
-		(effects
-			(font
-				(size 1.27 1.27)
-			)
-			(justify left bottom)
-		)
-	)
 	(label "USB_RP_D-"
 		(at 302.26 200.66 0)
@@
 	)
 	(symbol
-		(lib_id "DS_Capacitor_0402:1uF 50V 0402")
-		(at 92.71 109.22 0)
-		(mirror y)
-		(unit 1)
-		(exclude_from_sim no)
-		(in_bom yes)
-		(on_board yes)
-		(dnp no)
-		(property "Reference" "C54"
-			(at 88.9 106.6799 0)
-			(effects
-				(font
-					(size 1.27 1.27)
-				)
-				(justify left)
-			)
-		)
-		(property "Value" "1uF 50V"
-			(at 88.9 109.2199 0)
-			(effects
-				(font
-					(size 1.27 1.27)
-				)
-				(justify left)
-			)
-		)
-		(property "Footprint" "Capacitor_SMD:C_0402_1005Metric"
-			(at 88.9 113.284 0)
-			(show_name yes)
-			(effects
-				(font
-					(size 1.27 1.27)
-				)
-				(justify left)
-				(hide yes)
-			)
-		)
-		(property "Datasheet" ""
-			(at 88.9 117.348 0)
-			(show_name yes)
-			(effects
-				(font
-					(size 1.27 1.27)
-				)
-				(justify left)
-				(hide yes)
-			)
-		)
-		(property "Description" "50V 1uF X5R ±10% 0402 Multilayer Ceramic Capacitors MLCC - SMD/SMT ROHS"
-			(at 88.9 121.412 0)
-			(show_name yes)
-			(effects
-				(font
-					(size 1.27 1.27)
-				)
-				(justify left)
-				(hide yes)
-			)
-		)
-		(property "FOOTPRINT_SHORT" "0402"
-			(at 88.9 111.7599 0)
-			(effects
-				(font
-					(size 1.27 1.27)
-				)
-				(justify left)
-			)
-		)
-		(property "ROHS" "YES"
-			(at 88.9 123.444 0)
-			(show_name yes)
-			(effects
-				(font
-					(size 1.27 1.27)
-				)
-				(justify left)
-				(hide yes)
-			)
-		)
-		(property "LCSC_PART" "C1518208"
-			(at 88.9 115.316 0)
-			(show_name yes)
-			(effects
-				(font
-					(size 1.27 1.27)
-				)
-				(justify left)
-				(hide yes)
-			)
-		)
-		(property "MFR" ""
-			(at 88.9 119.38 0)
-			(show_name yes)
-			(effects
-				(font
-					(size 1.27 1.27)
-				)
-				(justify left)
-				(hide yes)
-			)
-		)
-		(pin "2"
-		)
-		(pin "1"
-		)
-		(instances
-			(project "PDNode_Baseboard"
-				(path "/f9e05184-c88b-4a88-ae9c-ab2bdb32be7c/c5103ceb-5325-4a84-a025-9638a412984e/2613c462-ed55-40aa-a079-4e429685a0a2"
-					(reference "C54")
-					(unit 1)
-				)
-			)
-		)
-	)
-	(symbol
 		(lib_id "DS_Supply:GND")
 		(at 266.7 218.44 0)
@@
 	)
 	(symbol
+		(lib_name "Green_0402_1")
 		(lib_id "DS_Opto:Green_0402")
 		(at 134.62 260.35 0)
@@
 	)
 	(symbol
+		(lib_name "5.1K 1% 0402_4")
 		(lib_id "DS_Resistor_0402:5.1K 1% 0402")
 		(at 130.81 203.2 0)
@@
 	)
 	(symbol
+		(lib_name "5.1K 1% 0402_3")
 		(lib_id "DS_Resistor_0402:5.1K 1% 0402")
 		(at 180.34 186.69 0)
@@
 	)
 	(symbol
+		(lib_name "100nF 50V 0402_2")
 		(lib_id "DS_Capacitor_0402:100nF 50V 0402")
 		(at 266.7 205.74 0)
@@
 	)
 	(symbol
+		(lib_name "100nF 50V 0402_3")
 		(lib_id "DS_Capacitor_0402:100nF 50V 0402")
 		(at 196.85 204.47 0)
@@
 	)
 	(symbol
+		(lib_name "5.1K 1% 0402_2")
 		(lib_id "DS_Resistor_0402:5.1K 1% 0402")
 		(at 180.34 204.47 0)
@@
 	)
 	(symbol
+		(lib_name "100nF 50V 0402_1")
 		(lib_id "DS_Capacitor_0402:100nF 50V 0402")
 		(at 260.35 97.79 0)
@@
 	)
 	(symbol
+		(lib_name "4.7uF 25V 0402_1")
+		(lib_id "DS_Capacitor_0402:4.7uF 25V 0402")
+		(at 92.71 109.22 0)
+		(mirror y)
+		(unit 1)
+		(exclude_from_sim no)
+		(in_bom yes)
+		(on_board yes)
+		(dnp no)
+		(property "Reference" "C54"
+			(at 88.9 106.6799 0)
+			(effects
+				(font
+					(size 1.27 1.27)
+				)
+				(justify left)
+			)
+		)
+		(property "Value" "4.7uF 25V"
+			(at 88.9 109.2199 0)
+			(effects
+				(font
+					(size 1.27 1.27)
+				)
+				(justify left)
+			)
+		)
+		(property "Footprint" "Capacitor_SMD:C_0402_1005Metric"
+			(at 88.9 113.284 0)
+			(show_name yes)
+			(effects
+				(font
+					(size 1.27 1.27)
+				)
+				(justify left)
+				(hide yes)
+			)
+		)
+		(property "Datasheet" ""
+			(at 88.9 117.348 0)
+			(show_name yes)
+			(effects
+				(font
+					(size 1.27 1.27)
+				)
+				(justify left)
+				(hide yes)
+			)
+		)
+		(property "Description" "25V 4.7uF X5R ±20% 0402 Multilayer Ceramic Capacitors MLCC - SMD/SMT ROHS"
+			(at 88.9 121.412 0)
+			(show_name yes)
+			(effects
+				(font
+					(size 1.27 1.27)
+				)
+				(justify left)
+				(hide yes)
+			)
+		)
+		(property "FOOTPRINT_SHORT" "0402"
+			(at 88.9 111.7599 0)
+			(effects
+				(font
+					(size 1.27 1.27)
+				)
+				(justify left)
+			)
+		)
+		(property "ROHS" "YES"
+			(at 88.9 123.444 0)
+			(show_name yes)
+			(effects
+				(font
+					(size 1.27 1.27)
+				)
+				(justify left)
+				(hide yes)
+			)
+		)
+		(property "LCSC_PART" "C22367824"
+			(at 88.9 115.316 0)
+			(show_name yes)
+			(effects
+				(font
+					(size 1.27 1.27)
+				)
+				(justify left)
+				(hide yes)
+			)
+		)
+		(property "MFR" "Murata"
+			(at 88.9 119.38 0)
+			(show_name yes)
+			(effects
+				(font
+					(size 1.27 1.27)
+				)
+				(justify left)
+				(hide yes)
+			)
+		)
+		(pin "2"
+		)
+		(pin "1"
+		)
+		(instances
+			(project "BladeCore-M54E"
+				(path "/f9e05184-c88b-4a88-ae9c-ab2bdb32be7c/c5103ceb-5325-4a84-a025-9638a412984e/2613c462-ed55-40aa-a079-4e429685a0a2"
+					(reference "C54")
+					(unit 1)
+				)
+			)
+		)
+	)
+	(symbol
 		(lib_id "DS_Resistor_1206:1M 1% 1206")
 		(at 54.61 223.52 90)
@@
 	)
 	(symbol
+		(lib_name "1K 1% 0402_1")
 		(lib_id "DS_Resistor_0402:1K 1% 0402")
 		(at 365.76 99.06 90)
@@
 	)
 	(symbol
+		(lib_name "5.1K 1% 0402_1")
 		(lib_id "DS_Resistor_0402:5.1K 1% 0402")
 		(at 118.11 203.2 0)
@@
 	)
 	(symbol
+		(lib_name "4.7uF 25V 0402_2")
 		(lib_id "DS_Capacitor_0402:4.7uF 25V 0402")
 		(at 143.51 195.58 0)
