File: src/HardwareDesign/1.0.0/usb_interface.kicad_sch (KiCad schematic)
At the start: 31 parts, among them IC7 TPS74801DRCT, IC8 SN74LVC1G97QDCKRQ1, IC9 FSUSB42MUX, J3 USB-TYPE-C-018

Commit message: export gerbers
Parts:
- removed D2: Green, LED_SMD:LED_0402_1005Metric, symbol DS_Opto:Green_0402
- removed R62: 1K 1%, Resistor_SMD:R_0402_1005Metric, symbol DS_Resistor_0402:1K 1% 0402
- added C60: 100nF 50V, Capacitor_SMD:C_0402_1005Metric, symbol DS_Capacitor_0402:100nF 50V 0402
- added D10, D11: Green, LED_SMD:LED_0402_1005Metric, symbol DS_Opto:Green_0402
- added D9: SS13, Diode_SMD:D_SMA, symbol Diode:SS13
- added IC10: SN74LVC1G97QDCKRQ1, DS_Peripherals:SOT-363_SC-70-6, symbol DS_Peripherals:SN74LVC1G97QDCKRQ1
- added R58, R61: 1K 1%, Resistor_SMD:R_0402_1005Metric, symbol DS_Resistor_0402:1K 1% 0402
- D8: now fitted; now in the parts list
Connections:
- net +3.3V: now also C60.1, IC10.3 (IN0), IC10.5 (VCC)
- net +5V: now also D9.2 (A); no longer C52.1, C53.1, C54.1, D4.1 (K), D8.1 (K), IC7.1 (IN), IC7.2 (IN), IC7.4 (BIAS), IC7.5 (EN)
- net GND: now also C60.2, IC10.2 (GND), R58.1, R61.2
- net USB_IND: now also D10.1, R58.2
- net VBUS: now also IC10.1 (IN1)
- net VBUS_ONBOARD: now also IC10.6 (IN2)
- new net: D11.1, R61.1
- new net: D11.2, IC10.4 (Y)
- new net REGIN: C52.1, C53.1, C54.1, D10.2, D4.1 (K), D8.1 (K), D9.1 (K), IC7.1 (IN), IC7.2 (IN), IC7.4 (BIAS), IC7.5 (EN)
Other:
- note added: "+5V INDICATOR LED"
- note added: "2-Input OR gate configuration"
- note added: "VBUS INDICATION LOGIC"
- note added: "VBUS_ONBOARD = 1 -> Y = 1 VBUS = 1 -> Y = 1"
- note removed: "If PGOOD AND PGOOD_3V3 are both 1, Y = 1"
- note removed: "USB INDICATOR LED"
- moved on the sheet: C57, C58, D6, IC8, IC9, R20, R60

Commit message: update documentation
Parts:
- C49, C50, C54: footprint Capacitor_SMD:C_0402_1005Metric -> DS_Capacitor:C_0402_1005Metric; DIST1 (none) -> https://de.farnell.com/en-DE/kyocera-avx/04023d475mat2a/cap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; MFR Murata -> KYOCERA AVX; MPN (none) -> 04023D475MAT2A
- C51, C52, C57, C58, C60: footprint Capacitor_SMD:C_0402_1005Metric -> DS_Capacitor:C_0402_1005Metric; DIST1 (none) -> https://de.farnell.com/en-DE/tdk/cga2b3x7r1h104k050bb/cap-0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; MFR (none) -> TDK; MPN (none) -> CGA2B3X7R1H104K050BB
- C53: footprint Capacitor_SMD:C_0402_1005Metric -> DS_Capacitor:C_0402_1005Metric; DIST1 (none) -> https://de.farnell.com/en-DE/murata/grm155r61h105ke05d/cap-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; MFR (none) -> Murata; MPN (none) -> GRM155R61H105KE05D
- C55: footprint Capacitor_SMD:C_0402_1005Metric -> DS_Capacitor:C_0402_1005Metric; DIST1 (none) -> https://de.farnell.com/en-DE/yageo/cc0402krx7r9bb222/cap-22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
- C56: footprint Capacitor_SMD:C_1206_3216Metric -> DS_Capacitor:C_1206_3216Metric; DIST1 (none) -> https://de.farnell.com/en-DE/samsung-electro-mechanics/cl31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
- C59: footprint Capacitor_SMD:C_1206_3216Metric -> DS_Capacitor:C_1206_3216Metric; DIST1 (none) -> https://de.farnell.com/en-DE/kemet/c1206x102kgractu/cap-100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; MFR Johanson Dielectrics -> KEMET; MPN (none) -> C1206X102KGRACTU
- D10, D11, D6: footprint LED_SMD:LED_0402_1005Metric -> DS_Opto:LED_0402_1005Metric
- D7: DIST1 (none) -> https://de.farnell.com/en-DE/littelfuse/sp0503bahtg/esd-pro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
- J3: DIST1 (none) -> https://de.farnell.com/en-DE/amphenol-communications-soluti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; DIST2 (none) -> https://www.digikey.de/en/products/detail/amphenol-cs-fci/1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; MFR DEALON -> Amphenol ICC (FCI); MPN USB-TYPE-C-018 -> 10171746-00021LF
- R19, R20, R52, R55, R56: footprint Resistor_SMD:R_0402_1005Metric -> DS_Resistor:R_0402_1005Metric; DIST1 (none) -> https://de.farnell.com/en-DE/vishay/crcw04025k10fked/res-5k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; MFR (none) -> VISHAY; MPN (none) -> CRCW04025K10FKED
- R53: footprint Resistor_SMD:R_0402_1005Metric -> DS_Resistor:R_0402_1005Metric; DIST1 (none) -> https://de.farnell.com/en-DE/vishay/crcw040210k0fked/res-10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; MFR ROHM -> VISHAY; MPN (none) -> CRCW040210K0FKED
- R54: footprint Resistor_SMD:R_0402_1005Metric -> DS_Resistor:R_0402_1005Metric; DIST1 (none) -> https://de.farnell.com/en-DE/vishay/crcw04027k50fked/res-7k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; MFR Uniohm -> VISHAY; MPN (none) -> CRCW04027K50FKED
- R57: footprint Resistor_SMD:R_1206_3216Metric -> DS_Resistor:R_1206_3216Metric; DIST1 (none) -> https://de.farnell.com/en-DE/vishay/crcw12061m00fkea/res-1m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; MPN (none) -> CRCW12061M00FKEA
- R58, R60, R61: footprint Resistor_SMD:R_0402_1005Metric -> DS_Resistor:R_0402_1005Metric; DIST1 (none) -> https://de.farnell.com/en-DE/vishay/crcw04021k00fked/res-1k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; MFR FH -> VISHAY; MPN (none) -> CRCW04021K00FKED
- R59: footprint Resistor_SMD:R_0402_1005Metric -> DS_Resistor:R_0402_1005Metric; DIST1 (none) -> https://de.farnell.com/en-DE/vishay/crcw04022k40fked/res-2k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; MFR LIZ -> VISHAY; MPN (none) -> CRCW04022K40FKED
