File: src/HardwareDesign/1.0.0/microcontroller.kicad_sch (KiCad schematic)
At the start: 32 parts, among them IC1 RP2354B

Commit message: add basic software
Connections:
- net USB_IND: no longer names the net of D3.1, R34.2
Changed lines of the file:
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@@
-		)
-	)
-	(label "USB_IND"
-		(at 121.92 254 0)
-		(effects
-			(font
-				(size 1.27 1.27)
-			)
-			(justify left bottom)
 		)
 	)
