File: src/HardwareDesign/1.0.0/microcontroller.kicad_sch (KiCad schematic)
At the start: 32 parts, among them IC1 RP2354B

Commit message: export gerbers
Connections:
- net HEARTBEAT: now also IC1.45 (GPIO36), R25.8 (R12); no longer R25.1 (R11)
- no-connect marks 0 -> 1
Changed lines of the file:
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@@
+	)
+	(junction
+		(at 245.11 109.22)
+		(diameter 0)
+		(color 0 0 0 0)
 	)
 	(junction
@@
 		(color 0 0 0 0)
 	)
+	(no_connect
+		(at 259.08 109.22)
+	)
 	(wire
 		(pts
@@
 	(wire
 		(pts
+			(xy 245.11 109.22) (xy 250.19 109.22)
+		)
+		(stroke
+			(width 0)
+			(type default)
+		)
+	)
+	(wire
+		(pts
 			(xy 154.94 66.04) (xy 175.26 66.04)
 		)
@@
 	(wire
 		(pts
-			(xy 245.11 109.22) (xy 250.19 109.22)
-		)
-		(stroke
-			(width 0)
-			(type default)
-		)
-	)
-	(wire
-		(pts
 			(xy 161.29 113.03) (xy 185.42 113.03)
 		)
@@
 	(wire
 		(pts
-			(xy 259.08 109.22) (xy 275.59 109.22)
-		)
-		(stroke
-			(width 0)
-			(type default)
-		)
-	)
-	(wire
-		(pts
 			(xy 127 144.78) (xy 146.05 144.78)
 		)
@@
 	(wire
 		(pts
+			(xy 245.11 105.41) (xy 275.59 105.41)
+		)
+		(stroke
+			(width 0)
+			(type default)
+		)
+	)
+	(wire
+		(pts
 			(xy 154.94 154.94) (xy 171.45 154.94)
 		)
@@
 	(wire
 		(pts
+			(xy 245.11 109.22) (xy 245.11 115.57)
+		)
+		(stroke
+			(width 0)
+			(type default)
+		)
+	)
+	(wire
+		(pts
 			(xy 237.49 97.79) (xy 219.71 97.79)
 		)
@@
 	(wire
 		(pts
-			(xy 245.11 109.22) (xy 245.11 115.57)
+			(xy 245.11 105.41) (xy 245.11 109.22)
 		)
 		(stroke
@@
 	(global_label "HEARTBEAT"
 		(shape input)
-		(at 275.59 109.22 0)
+		(at 275.59 105.41 0)
 		(fields_autoplaced yes)
 		(effects
@@
 		)
 		(property "Intersheetrefs" "${INTERSHEET_REFS}"
-			(at 288.8561 109.22 0)
+			(at 288.8561 105.41 0)
 			(effects
 				(font

Commit message: update documentation
Parts:
- C25, C26, C27, C28, C29, C30, C31, C32: footprint Capacitor_SMD:C_0402_1005Metric -> DS_Capacitor:C_0402_1005Metric; DIST1 (none) -> https://de.farnell.com/en-DE/samsung-electro-mechanics/cl05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; MFR (none) -> Samsung; MPN (none) -> CL05B102KB5NNNC
- D3: footprint LED_SMD:LED_0402_1005Metric -> DS_Opto:LED_0402_1005Metric; DIST1 (none) -> https://de.farnell.com/en-DE/qt-brightek/qblp595-2ib5/led-b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; MFR XINGLIGHT -> QT BRIGHTEK; MPN XL-1005UBC -> QBLP595-2IB5
- IC1: DIST1 (none) -> https://www.digikey.de/en/products/detail/raspberry-pi/SC15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
- R12, R14, R21, R26, R29, R31, R32, R33: footprint Resistor_SMD:R_0402_1005Metric -> DS_Resistor:R_0402_1005Metric; DIST1 (none) -> https://de.farnell.com/en-DE/vishay/crcw0402100rfked/res-10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; MFR (none) -> VISHAY; MPN (none) -> CRCW0402100RFKED
- R13, R15, R16, R22, R23, R24, R25, R27, R28, R30: footprint Resistor_SMD:R_Array_Convex_4x0603 -> DS_Resistor:R_Array_Convex_4x0603
- R17, R18: footprint Resistor_SMD:R_0402_1005Metric -> DS_Resistor:R_0402_1005Metric; DIST1 (none) -> https://de.farnell.com/en-DE/vishay/crcw04022k20fked/res-2k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; MFR (none) -> VISHAY; MPN (none) -> CRCW04022K20FKED
- R34: footprint Resistor_SMD:R_0402_1005Metric -> DS_Resistor:R_0402_1005Metric; DIST1 (none) -> https://de.farnell.com/en-DE/vishay/crcw04021k00fked/res-1k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; MFR FH -> VISHAY; MPN (none) -> CRCW04021K00FKED
