File: src/HardwareDesign/1.0.0/BladeCore-M54E.kicad_pcb (KiCad board)
At the start: 6 copper layers, 29 x 80.6 mm, 146 parts, among them IC1 RP2354B, IC2 AT24C256C-XHL-T, IC3 W25Q128JVPIQ, IC4 MCP6001RT, IC5 LM4040B30FTA, IC6 W5500, IC7 TPS74801DRCT, IC8 SN74LVC1G97QDCKRQ1, IC9 FSUSB42MUX, J1 MDT320M03001, J2 SM03B-SRSS-TB, J3 USB-TYPE-C-018, SW1 B3U-1000P, SW2 B3U-1000P, X1 12MHz 10pF, X2 25MHz 12pF

Commit message: update design
Parts:
- C54: value 1uF 50V -> 4.7uF 25V
Connections:
- C54 pad 1: /Project Architecture/USB Interface and Power/BIAS -> +5V
- IC7 pad 4: /Project Architecture/USB Interface and Power/BIAS -> +5V
- J1 pad SH1: (no net) -> GND
Routing:
- net /Project Architecture/PWR: track 114.1 -> 116.5 mm, vias 6 -> 4
- net +5V: track 73.3 -> 75.0 mm
- net /Project Architecture/USB Interface and Power/BIAS: track 1.38 -> 0.00 mm
- net GND: track 237.9 -> 237.6 mm, vias 158 -> 163
Other:
- board text added: "HWREV 1.0.0"

Commit message: add basic software
Connections:
- net /Project Architecture/Microcontroller/USB_IND renamed Net-(D3-Pad1)
- J1 pad SH1: GND -> (no net)
Changed lines of the file:
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@@
 	(net 29 "QSPI_SD1")
 	(net 30 "/Project Architecture/USB Interface and Power/USB_IND")
-	(net 31 "/Project Architecture/Microcontroller/USB_IND")
+	(net 31 "Net-(D3-Pad1)")
 	(net 32 "QSPI_SS")
 	(net 33 "/Project Architecture/Microcontroller Peripherals/RP_D-")
@@
 			)
 		)
-		(property "Datasheet" "~"
+		(property "Datasheet" ""
 			(at 0 0 270)
 			(unlocked yes)
@@
 			(layers "F.Cu" "F.Mask" "F.Paste")
 			(roundrect_rratio 0.25)
-			(net 31 "/Project Architecture/Microcontroller/USB_IND")
+			(net 31 "Net-(D3-Pad1)")
 			(pintype "passive")
 		)
@@
 			(layers "*.Cu" "*.Mask")
 			(remove_unused_layers no)
-			(net 1 "GND")
 		)
 		(embedded_fonts no)
@@
 			(layers "F.Cu" "F.Mask" "F.Paste")
 			(roundrect_rratio 0.25)
-			(net 31 "/Project Architecture/Microcontroller/USB_IND")
+			(net 31 "Net-(D3-Pad1)")
 			(pintype "passive")
 		)

Commit message: export gerbers
Parts:
- removed D2: Green, LED_SMD:LED_0402_1005Metric
- removed JP1: SolderJumper_3_Open, Jumper:SolderJumper-3_P1.3mm_Open_RoundedPad1.0x1.5mm
- removed R62: 1K 1%, Resistor_SMD:R_0402_1005Metric
- added C60: 100nF 50V, Capacitor_SMD:C_0402_1005Metric, B.Cu at (210.1, 140.4)
- added D10: Green, LED_SMD:LED_0402_1005Metric, F.Cu at (208.8, 99.1)
- added D11: Green, LED_SMD:LED_0402_1005Metric, F.Cu at (211.0, 85.9)
- added D9: SS13, Diode_SMD:D_SMA, B.Cu at (209.1, 145.8)
- added IC10: SN74LVC1G97QDCKRQ1, DS_Peripherals:SOT-363_SC-70-6, B.Cu at (210.4, 138.0)
- added R58: 1K 1%, Resistor_SMD:R_0402_1005Metric, F.Cu at (208.8, 101.3)
- added R61: 1K 1%, Resistor_SMD:R_0402_1005Metric, F.Cu at (211.5, 87.6)
- moved D4 0.05 mm to (209.1, 145.8)
Connections:
- C52 pad 1: +5V -> REGIN
- C53 pad 1: +5V -> REGIN
- C54 pad 1: +5V -> REGIN
- D4 pad 1: +5V -> REGIN
- D8 pad 1: +5V -> REGIN
- IC1 pad 45: Net-(IC1B-GPIO36) -> HEARTBEAT
- IC7 pad 1: +5V -> REGIN
- IC7 pad 2: +5V -> REGIN
- IC7 pad 4: +5V -> REGIN
- IC7 pad 5: +5V -> REGIN
- J1 pad 10: /Project Architecture/PWR -> +3.3V
- J1 pad 12: /Project Architecture/PWR -> +3.3V
- J1 pad 14: /Project Architecture/PWR -> +5V
- J1 pad 16: /Project Architecture/PWR -> +5V
- R25 pad 1: HEARTBEAT -> unconnected-(R25-R11-Pad1)
- R25 pad 8: Net-(IC1B-GPIO36) -> HEARTBEAT
Routing:
- net /Project Architecture/PWR: track 116.5 -> 0.00 mm, vias 4 -> 0
- net REGIN: track 0.00 -> 75.9 mm, vias 0 -> 12
- net Net-(IC10-Y): track 0.00 -> 55.8 mm, vias 0 -> 3
- net VBUS: track 94.3 -> 40.5 mm, vias 6 -> 5
- net VBUS_ONBOARD: track 48.7 -> 87.8 mm
- net +5V: track 75.0 -> 46.3 mm, vias 11 -> 5
- net +3.3V: track 50.2 -> 68.0 mm, vias 41 -> 44
- net GND: track 237.6 -> 243.9 mm, vias 163 -> 164
- net Net-(IC1B-GPIO36): track 2.53 -> 0.00 mm
- net /Project Architecture/Microcontroller Peripherals/I2C0_SDA: track 21.9 -> 19.8 mm
- net /Project Architecture/Microcontroller Peripherals/I2C0_SCL: track 20.8 -> 18.7 mm
- net Net-(D11-Pad1): track 0.00 -> 1.22 mm
- net VBUS_ISO: track 2.95 -> 2.43 mm
- added copper zone on B.Cu, net REGIN
- added copper zone on F.Cu, net REGIN
- added copper zone on In3.Cu, net REGIN
- removed copper zone on B.Cu, net +5V
- removed copper zone on F.Cu, net +5V
- removed copper zone on In3.Cu, net +5V
Other:
- board text added: "REG_ON"
- board text removed: "3V3"
- board text removed: "5V"

Commit message: update documentation
Parts:
- C1, C10, C11, C12, C13, C14, C15, C16, C17, C18, C19, C2, C20, C21, C22, C23, C24, C25, C26, C27, C28, C29, C3, C30, C31, C32, C33, C34, C35, C36, C37, C38, C39, C4, C40, C41, C42, C43, C44, C45, C46, C47, C48, C49, C5, C50, C51, C52, C53, C54, C55, C57, C58, C6, C60, C7, C8, C9: footprint Capacitor_SMD:C_0402_1005Metric -> DS_Capacitor:C_0402_1005Metric
- C56, C59: footprint Capacitor_SMD:C_1206_3216Metric -> DS_Capacitor:C_1206_3216Metric
- D10, D11, D3, D6: footprint LED_SMD:LED_0402_1005Metric -> DS_Opto:LED_0402_1005Metric
- J1: footprint DS_Connector:M.2-M-KEY_Card_2280 -> DS_Connector:M.2-M-KEY_Card_Plain
- R1, R10, R11, R12, R14, R17, R18, R19, R2, R20, R21, R26, R29, R3, R31, R32, R33, R34, R35, R36, R37, R38, R39, R4, R40, R41, R42, R43, R44, R45, R46, R47, R48, R49, R5, R50, R52, R53, R54, R55, R56, R58, R59, R6, R60, R61, R7, R8, R9: footprint Resistor_SMD:R_0402_1005Metric -> DS_Resistor:R_0402_1005Metric
- R13, R15, R16, R22, R23, R24, R25, R27, R28, R30: footprint Resistor_SMD:R_Array_Convex_4x0603 -> DS_Resistor:R_Array_Convex_4x0603
- R51, R57: footprint Resistor_SMD:R_1206_3216Metric -> DS_Resistor:R_1206_3216Metric
- moved J1 39.1 mm to (221.4, 164.6)
Connections:
- IC5 pad 3: (no net) -> unconnected-(IC5-NC-Pad3)
Routing:
- net GND: track 243.9 -> 244.0 mm, vias 164 -> 165
