File: src/HardwareDesign/1.0.0/Project Architecture.kicad_sch (KiCad schematic)
At the start: 4 parts, among them J1 MDT320M03001

Commit message: export gerbers
Parts:
- removed JP1: SolderJumper_3_Open, Jumper:SolderJumper-3_P1.3mm_Open_RoundedPad1.0x1.5mm, symbol Jumper:SolderJumper_3_Open
- R51: now fitted; now in the parts list
Connections:
- net +3.3V: now also J1.10, J1.12
- net +5V: now also J1.14, J1.16
- removed net PWR: J1.10, J1.12, J1.14, J1.16
Other:
- note removed: "R37 + R38 (5.1 kΩ) + C21 (100 nF): VBUS voltage sense divider and RC filtering for the ADC input; with equal resistors the ADC sees VBUS/2. Only USB-Attached detection"

Commit message: update documentation
Parts:
- removed J1: MDT320M03001, DS_Connector:M.2-M-KEY_Card_2280, symbol DS_Connector:PCIe M.2 M-Key Card
- added J1: MDT320M03001, DS_Connector:M.2-M-KEY_Card_Plain, symbol DS_Connector:PCIe M.2 M-Key Card_Plain
- D5: DIST1 (none) -> https://de.farnell.com/en-DE/littelfuse/sp0503bahtg/esd-pro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
- R51: footprint Resistor_SMD:R_1206_3216Metric -> DS_Resistor:R_1206_3216Metric; LCSC_PART C205296 -> C17888
Connections:
- net +3.3V: now also J1.10, J1.12
- net +5V: now also J1.14, J1.16
- net ACT_LED: now also J1.20
- net ADC0: now also J1.46
- net ADC1: now also J1.48
- net ADC2: now also J1.50
- net ADC3: now also J1.52
- net ADC4: now also J1.54
- net ADC5: now also J1.56
- net GND: now also J1.1, J1.11, J1.2, J1.22, J1.23, J1.26, J1.32, J1.38, J1.41, J1.42, J1.44, J1.58, J1.67, J1.68, J1.70, J1.73, J1.S1 (SHIELD)
- net GPIO0: now also J1.57
- net GPIO1: now also J1.55
- net GPIO10: now also J1.35
- net GPIO11: now also J1.33
- net GPIO12: now also J1.31
- net GPIO13: now also J1.29
- net GPIO14: now also J1.27
- net GPIO15: now also J1.25
- net GPIO16: now also J1.21
- net GPIO17: now also J1.19
- net GPIO18: now also J1.17
- net GPIO19: now also J1.15
- net GPIO2: now also J1.53
- net GPIO20: now also J1.13
- net GPIO21: now also J1.9
- net GPIO22: now also J1.7
- net GPIO23: now also J1.5
- net GPIO24: now also J1.3
- net GPIO25: now also J1.8
- net GPIO26: now also J1.6
- net GPIO27: now also J1.4
- net GPIO3: now also J1.51
- net GPIO4: now also J1.49
- net GPIO5: now also J1.47
- net GPIO6: now also J1.45
- net GPIO7: now also J1.43
- net GPIO8: now also J1.39
- net GPIO9: now also J1.37
- net LINK_LED: now also J1.18
- net RCT: now also J1.24
- net RD_N: now also J1.30
- net RD_P: now also J1.28
- net TCT: now also J1.40
- net TD_N: now also J1.36
- net TD_P: now also J1.34
- net USB_D+: now also J1.69
- net USB_D-: now also J1.71
- net VBUS: now also J1.72, J1.74, J1.75
