File: src/HardwareDesign/1.0.0/ethernet_interface.kicad_sch (KiCad schematic)
At the start: 35 parts, among them IC6 W5500, X2 25MHz 12pF

Commit message: update documentation
Parts:
- C33, C34: footprint Capacitor_SMD:C_0402_1005Metric -> DS_Capacitor:C_0402_1005Metric; DIST1 (none) -> https://de.farnell.com/en-DE/kemet/c0402c682k5ractu/cap-680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; MFR (none) -> KEMET; MPN (none) -> C0402C682K5RACTU
- C35, C36: footprint Capacitor_SMD:C_0402_1005Metric -> DS_Capacitor:C_0402_1005Metric; DIST1 (none) -> https://de.farnell.com/en-DE/yageo/cc0402jrnpo9bn150/cap-15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; MFR (none) -> YAGEO; MPN (none) -> CC0402JRNPO9BN150
- C37, C38, C40, C41, C42, C43, C44, C45, C46, C47, C48: footprint Capacitor_SMD:C_0402_1005Metric -> DS_Capacitor:C_0402_1005Metric; DIST1 (none) -> https://de.farnell.com/en-DE/tdk/cga2b3x7r1h104k050bb/cap-0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; MFR (none) -> TDK; MPN (none) -> CGA2B3X7R1H104K050BB
- C39: footprint Capacitor_SMD:C_0402_1005Metric -> DS_Capacitor:C_0402_1005Metric; DIST1 (none) -> https://de.farnell.com/en-DE/kyocera-avx/04023d475mat2a/cap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; MFR Murata -> KYOCERA AVX; MPN (none) -> 04023D475MAT2A
- IC6: DIST1 (none) -> https://www.digikey.de/en/products/detail/wiznet/W5500/4425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
- L2: DIST1 (none) -> https://de.farnell.com/en-DE/murata/blm18he152sn1d/ferrite-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; ROHS (none) -> YES
- R35: footprint Resistor_SMD:R_0402_1005Metric -> DS_Resistor:R_0402_1005Metric; DIST1 (none) -> https://de.farnell.com/en-DE/vishay/crcw04024k70fked/res-4k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; MFR (none) -> VISHAY; MPN (none) -> CRCW04024K70FKED
- R36, R45, R47: footprint Resistor_SMD:R_0402_1005Metric -> DS_Resistor:R_0402_1005Metric; DIST1 (none) -> https://de.farnell.com/en-DE/vishay/crcw0402470rfked/res-47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; MFR Panasonic -> VISHAY; MPN (none) -> CRCW0402470RFKED
- R37, R38, R48, R49: footprint Resistor_SMD:R_0402_1005Metric -> DS_Resistor:R_0402_1005Metric; DIST1 (none) -> https://de.farnell.com/en-DE/vishay/crcw040249r9fked/res-49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; MFR (none) -> VISHAY; MPN (none) -> CRCW040249R9FKED
- R39, R41, R44, R46: footprint Resistor_SMD:R_0402_1005Metric -> DS_Resistor:R_0402_1005Metric; DIST1 (none) -> https://de.farnell.com/en-DE/vishay/crcw04023r30fked/res-3r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; MFR (none) -> VISHAY; MPN (none) -> CRCW04023R30FKED
- R40, R42: footprint Resistor_SMD:R_0402_1005Metric -> DS_Resistor:R_0402_1005Metric; DIST1 (none) -> https://de.farnell.com/en-DE/vishay/rca04020000zsed/res-0r0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; MFR YAGEO -> VISHAY; MPN (none) -> RCA04020000ZSED
- R43: footprint Resistor_SMD:R_0402_1005Metric -> DS_Resistor:R_0402_1005Metric; DIST1 (none) -> https://de.farnell.com/en-DE/vishay/crcw04021m00fked/res-1m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; MFR Vishay -> VISHAY; MPN (none) -> CRCW04021M00FKED
- R50: footprint Resistor_SMD:R_0402_1005Metric -> DS_Resistor:R_0402_1005Metric; DIST1 (none) -> https://de.farnell.com/en-DE/vishay/crcw040212k4fkedc/res-1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; MFR (none) -> VISHAY; MPN (none) -> CRCW040212K4FKEDC
- X2: DIST1 (none) -> https://de.farnell.com/en-DE/abracon/abm8aig-25-000mhz-12-2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; MFR YXC Crystal Oscillators -> ABRACON; MPN X322525MOB4SI -> ABM8AIG-25.000MHZ-12-2Z-T3
