File: src/HardwareDesign/1.0.0/microcontroller_peripherals.kicad_sch (KiCad schematic)
At the start: 45 parts, among them IC1 RP2354B, IC2 AT24C256C-XHL-T, IC3 W25Q128JVPIQ, IC4 MCP6001RT, IC5 LM4040B30FTA, J2 SM03B-SRSS-TB, SW1 B3U-1000P, SW2 B3U-1000P, X1 12MHz 10pF

Commit message: update documentation
Parts:
- C1, C10, C13, C14, C15, C17, C18, C19, C2, C21, C23, C3, C4, C5, C7, C8, C9: footprint Capacitor_SMD:C_0402_1005Metric -> DS_Capacitor:C_0402_1005Metric; DIST1 (none) -> https://de.farnell.com/en-DE/tdk/cga2b3x7r1h104k050bb/cap-0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; MFR (none) -> TDK; MPN (none) -> CGA2B3X7R1H104K050BB
- C11, C12: footprint Capacitor_SMD:C_0402_1005Metric -> DS_Capacitor:C_0402_1005Metric; DIST1 (none) -> https://de.farnell.com/en-DE/kemet/c0402h100j5gact500/capac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; MFR CCTC -> KEMET; MPN (none) -> C0402H100J5GACT500
- C16, C6: footprint Capacitor_SMD:C_0402_1005Metric -> DS_Capacitor:C_0402_1005Metric; DIST1 (none) -> https://de.farnell.com/en-DE/kyocera-avx/04023d475mat2a/cap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; MFR Murata -> KYOCERA AVX; MPN (none) -> 04023D475MAT2A
- C20, C22, C24: footprint Capacitor_SMD:C_0402_1005Metric -> DS_Capacitor:C_0402_1005Metric; DIST1 (none) -> https://de.farnell.com/en-DE/samsung-electro-mechanics/cl05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; MFR (none) -> Samsung; MPN (none) -> CL05A475KP5NRNC
- IC1: DIST1 (none) -> https://www.digikey.de/en/products/detail/raspberry-pi/SC15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
- IC3: DIST1 (none) -> https://www.digikey.de/en/products/detail/winbond-electroni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
- L1: DIST1 (none) -> https://de.farnell.com/en-DE/abracon/aota-b201610s3r3-101-t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; DIST2 (none) -> https://www.digikey.de/short/qdbv4bnm
- R1, R8: footprint Resistor_SMD:R_0402_1005Metric -> DS_Resistor:R_0402_1005Metric; DIST1 (none) -> https://de.farnell.com/en-DE/vishay/crcw04024k70fked/res-4k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; MFR (none) -> VISHAY; MPN (none) -> CRCW04024K70FKED
- R10, R11: footprint Resistor_SMD:R_0402_1005Metric -> DS_Resistor:R_0402_1005Metric; DIST1 (none) -> https://de.farnell.com/en-DE/vishay/crcw040210k0fked/res-10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; MFR ROHM -> VISHAY; MPN (none) -> CRCW040210K0FKED
- R2, R3, R4: footprint Resistor_SMD:R_0402_1005Metric -> DS_Resistor:R_0402_1005Metric; DIST1 (none) -> https://de.farnell.com/en-DE/vishay/crcw040233r0fked/res-33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; MFR ROHM -> VISHAY; MPN (none) -> CRCW040233R0FKED
- R5, R6: footprint Resistor_SMD:R_0402_1005Metric -> DS_Resistor:R_0402_1005Metric; DIST1 (none) -> https://de.farnell.com/en-DE/vishay/crcw04021k00fked/res-1k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; MFR FH -> VISHAY; MPN (none) -> CRCW04021K00FKED
- R7, R9: footprint Resistor_SMD:R_0402_1005Metric -> DS_Resistor:R_0402_1005Metric; DIST1 (none) -> https://de.farnell.com/en-DE/vishay/crcw040227r0fked/res-27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; MFR (none) -> VISHAY; MPN (none) -> CRCW040227R0FKED
- SW1, SW2: DIST1 (none) -> https://de.farnell.com/en-DE/omron/b3u-1000p/switch-spst-no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
- X1: DIST1 (none) -> https://de.farnell.com/en-DE/abracon/abm8g-12-000mhz-b4y-t/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; LCSC_PART C20625731 -> C2901649; MFR YXC Crystal Oscillators -> ABRACON; MPN ABM8-272-T3 -> ABM8G-12.000MHZ-B4Y-T
